Commit message: feat(robot_description): upgrade tank caterpillar track dynamics and 3d lidar simulation

File: robot_description/urdf/robot_core.xacro (robot description, xacro)
@@ -1,36 +1,50 @@
 <?xml version="1.0"?>
 <robot xmlns:xacro="http://www.ros.org/wiki/xacro">
-    <material name="dark_grey"><color rgba="0.20 0.21 0.23 1.0"/></material>
-    <material name="mid_grey"><color rgba="0.50 0.53 0.57 1.0"/></material>
+    <material name="dark_grey"><color rgba="0.18 0.19 0.21 1.0"/></material>
+    <material name="mid_grey"><color rgba="0.45 0.48 0.52 1.0"/></material>
     <material name="light_grey"><color rgba="0.78 0.80 0.82 1.0"/></material>
-    <material name="black"><color rgba="0.05 0.05 0.05 1.0"/></material>
-    <material name="accent_orange"><color rgba="0.82 0.52 0.18 1.0"/></material>
+    <material name="black"><color rgba="0.04 0.04 0.04 1.0"/></material>
+    <material name="accent_orange"><color rgba="0.85 0.50 0.15 1.0"/></material>
     <material name="green_pcb"><color rgba="0.13 0.55 0.13 1.0"/></material>
+    <material name="tread_dark"><color rgba="0.08 0.08 0.09 1.0"/></material>
+    <material name="tank_armor"><color rgba="0.24 0.25 0.27 1.0"/></material>
     <xacro:macro name="turtlebot_core">
         <xacro:property name="PI" value="3.1415926535897931" />
-        <xacro:property name="base_x" value="0.281" />
-        <xacro:property name="base_y" value="0.306" />
-        <xacro:property name="base_z" value="0.070" />
-        <xacro:property name="base_mass" value="1.80" />
-        <xacro:property name="wheel_radius" value="0.033" />
-        <xacro:property name="wheel_width" value="0.018" />
-        <xacro:property name="wheel_mass" value="0.05" />
-        <xacro:property name="wheel_separation" value="0.287" />
-        <xacro:property name="wheel_x_offset" value="0.0" />
-        <xacro:property name="caster_radius" value="0.008" />
-        <xacro:property name="caster_mass" value="0.01" />
+        <!-- Chassis dimensions (Armored Tank style) -->
+        <xacro:property name="base_x" value="0.300" />
+        <xacro:property name="base_y" value="0.200" />
+        <xacro:property name="base_z" value="0.080" />
+        <xacro:property name="base_mass" value="7.00" />
+        <!-- Tank Track Dimensions -->
+        <xacro:property name="track_y_offset" value="0.135" /> <!-- Center of track: y = +/- 0.135 m -->
+        <xacro:property name="track_width" value="0.046" />
+        <xacro:property name="track_separation" value="0.270" /> <!-- 2 * track_y_offset -->
+        <!-- Road Wheels (3 per side) -->
+        <xacro:property name="road_radius" value="0.045" />
+        <xacro:property name="road_width" value="0.044" />
+        <xacro:property name="road_mass" value="0.06" />
+        <!-- Front Sprocket & Rear Idler (Raised for climbing) -->
+        <xacro:property name="sprocket_radius" value="0.038" />
+        <xacro:property name="sprocket_width" value="0.044" />
+        <xacro:property name="sprocket_mass" value="0.05" />
+        <xacro:property name="sprocket_x" value="0.142" />
+        <xacro:property name="sprocket_z" value="0.016" />
+        <!-- Top plate & standoffs for sensors -->
         <xacro:property name="standoff_radius" value="0.008" />
-        <xacro:property name="standoff_height" value="0.108" />
-        <xacro:property name="plate_x" value="0.230" />
-        <xacro:property name="plate_y" value="0.230" />
+        <xacro:property name="standoff_height" value="0.095" />
+        <xacro:property name="plate_x" value="0.260" />
+        <xacro:property name="plate_y" value="0.200" />
         <xacro:property name="plate_z" value="0.006" />
-        <xacro:property name="plate_mass" value="0.15" />
+        <xacro:property name="plate_mass" value="0.20" />
+        <!-- Base Footprint: Projected on the ground plane -->
         <link name="base_footprint" />
         <joint name="base_footprint_joint" type="fixed">
             <parent link="base_footprint" />
             <child link="base_link" />
-            <origin xyz="0.0 0.0 ${wheel_radius}" rpy="0 0 0" />
+            <origin xyz="0.0 0.0 ${road_radius}" rpy="0 0 0" />
         </joint>
+        <!-- Base Link: Heavy-Duty Tank Chassis with Integrated Caterpillar Track Belts -->
         <link name="base_link">
+            <!-- Main Armored Hull -->
             <visual>
                 <origin xyz="0.0 0.0 ${base_z/2}" rpy="0 0 0" />
@@ -38,28 +52,237 @@
                     <box size="${base_x} ${base_y} ${base_z}" />
                 </geometry>
-                <material name="dark_grey" />
-            </visual>
+                <material name="tank_armor" />
+            </visual>
+            <!-- Front Sloped Glacis Armor Plate -->
+            <visual>
+                <origin xyz="${base_x/2 - 0.015} 0.0 ${base_z/2}" rpy="0 0.65 0" />
+                <geometry>
+                    <box size="0.050 ${base_y - 0.004} ${base_z - 0.004}" />
+                </geometry>
+                <material name="accent_orange" />
+            </visual>
+            <!-- ================= LEFT TANK TRACK VISUALS ================= -->
+            <!-- Left Track: Bottom Flat Belt (ground contact) -->
+            <visual>
+                <origin xyz="0.0 ${track_y_offset} ${-road_radius + 0.004}" rpy="0 0 0" />
+                <geometry>
+                    <box size="0.150 ${track_width} 0.008" />
+                </geometry>
+                <material name="tread_dark" />
+            </visual>
+            <!-- Left Track: Top Flat Belt -->
+            <visual>
+                <origin xyz="0.0 ${track_y_offset} ${sprocket_z + sprocket_radius - 0.004}" rpy="0 0 0" />
+                <geometry>
+                    <box size="0.284 ${track_width} 0.008" />
+                </geometry>
+                <material name="tread_dark" />
+            </visual>
+            <!-- Left Track: Front Climbing Slope -->
+            <visual>
+                <origin xyz="0.108 ${track_y_offset} 0.005" rpy="0 -0.85 0" />
+                <geometry>
+                    <box size="0.114 ${track_width} 0.008" />
+                </geometry>
+                <material name="tread_dark" />
+            </visual>
+            <!-- Left Track: Rear Slope -->
+            <visual>
+                <origin xyz="-0.108 ${track_y_offset} 0.005" rpy="0 0.85 0" />
+                <geometry>
+                    <box size="0.114 ${track_width} 0.008" />
+                </geometry>
+                <material name="tread_dark" />
+            </visual>
+            <!-- Left Track: Front Nose Cap -->
+            <visual>
+                <origin xyz="${sprocket_x} ${track_y_offset} ${sprocket_z}" rpy="${PI/2} 0 0" />
+                <geometry>
+                    <cylinder radius="${sprocket_radius + 0.002}" length="${track_width}" />
+                </geometry>
+                <material name="tread_dark" />
+            </visual>
+            <!-- Left Track: Rear Tail Cap -->
+            <visual>
+                <origin xyz="${-sprocket_x} ${track_y_offset} ${sprocket_z}" rpy="${PI/2} 0 0" />
+                <geometry>
+                    <cylinder radius="${sprocket_radius + 0.002}" length="${track_width}" />
+                </geometry>
+                <material name="tread_dark" />
+            </visual>
+            <!-- Left Track: Cleats / Grousers on Top Belt -->
+            <visual><origin xyz="-0.120 ${track_y_offset} ${sprocket_z + sprocket_radius + 0.002}" rpy="0 0 0" /><geometry><box size="0.008 ${track_width + 0.002} 0.004" /></geometry><material name="black" /></visual>
+            <visual><origin xyz="-0.085 ${track_y_offset} ${sprocket_z + sprocket_radius + 0.002}" rpy="0 0 0" /><geometry><box size="0.008 ${track_width + 0.002} 0.004" /></geometry><material name="black" /></visual>
+            <visual><origin xyz="-0.050 ${track_y_offset} ${sprocket_z + sprocket_radius + 0.002}" rpy="0 0 0" /><geometry><box size="0.008 ${track_width + 0.002} 0.004" /></geometry><material name="black" /></visual>
+            <visual><origin xyz="-0.017 ${track_y_offset} ${sprocket_z + sprocket_radius + 0.002}" rpy="0 0 0" /><geometry><box size="0.008 ${track_width + 0.002} 0.004" /></geometry><material name="black" /></visual>
+            <visual><origin xyz="0.017 ${track_y_offset} ${sprocket_z + sprocket_radius + 0.002}" rpy="0 0 0" /><geometry><box size="0.008 ${track_width + 0.002} 0.004" /></geometry><material name="black" /></visual>
+            <visual><origin xyz="0.050 ${track_y_offset} ${sprocket_z + sprocket_radius + 0.002}" rpy="0 0 0" /><geometry><box size="0.008 ${track_width + 0.002} 0.004" /></geometry><material name="black" /></visual>
+            <visual><origin xyz="0.085 ${track_y_offset} ${sprocket_z + sprocket_radius + 0.002}" rpy="0 0 0" /><geometry><box size="0.008 ${track_width + 0.002} 0.004" /></geometry><material name="black" /></visual>
+            <visual><origin xyz="0.120 ${track_y_offset} ${sprocket_z + sprocket_radius + 0.002}" rpy="0 0 0" /><geometry><box size="0.008 ${track_width + 0.002} 0.004" /></geometry><material name="black" /></visual>
+            <!-- Left Track: Mudguard / Fender -->
+            <visual>
+                <origin xyz="0.0 ${track_y_offset} 0.060" rpy="0 0 0" />
+                <geometry>
+                    <box size="0.300 ${track_width + 0.010} 0.004" />
+                </geometry>
+                <material name="mid_grey" />
+            </visual>
+            <visual>
+                <origin xyz="0.165 ${track_y_offset} 0.050" rpy="0 0.50 0" />
+                <geometry>
+                    <box size="0.045 ${track_width + 0.010} 0.004" />
+                </geometry>
+                <material name="mid_grey" />
+            </visual>
+            <visual>
+                <origin xyz="-0.165 ${track_y_offset} 0.050" rpy="0 -0.50 0" />
+                <geometry>
+                    <box size="0.045 ${track_width + 0.010} 0.004" />
+                </geometry>
+                <material name="mid_grey" />
+            </visual>
+            <visual>
+                <origin xyz="0.0 ${track_y_offset + track_width/2 + 0.004} 0.048" rpy="0 0 0" />
+                <geometry>
+                    <box size="0.280 0.003 0.020" />
+                </geometry>
+                <material name="mid_grey" />
+            </visual>
+            <!-- ================= RIGHT TANK TRACK VISUALS ================= -->
+            <!-- Right Track: Bottom Flat Belt -->
+            <visual>
+                <origin xyz="0.0 ${-track_y_offset} ${-road_radius + 0.004}" rpy="0 0 0" />
+                <geometry>
+                    <box size="0.150 ${track_width} 0.008" />
+                </geometry>
+                <material name="tread_dark" />
+            </visual>
+            <!-- Right Track: Top Flat Belt -->
+            <visual>
+                <origin xyz="0.0 ${-track_y_offset} ${sprocket_z + sprocket_radius - 0.004}" rpy="0 0 0" />
+                <geometry>
+                    <box size="0.284 ${track_width} 0.008" />
+                </geometry>
+                <material name="tread_dark" />
+            </visual>
+            <!-- Right Track: Front Climbing Slope -->
+            <visual>
+                <origin xyz="0.108 ${-track_y_offset} 0.005" rpy="0 -0.85 0" />
+                <geometry>
+                    <box size="0.114 ${track_width} 0.008" />
+                </geometry>
+                <material name="tread_dark" />
+            </visual>
+            <!-- Right Track: Rear Slope -->
+            <visual>
+                <origin xyz="-0.108 ${-track_y_offset} 0.005" rpy="0 0.85 0" />
+                <geometry>
+                    <box size="0.114 ${track_width} 0.008" />
+                </geometry>
+                <material name="tread_dark" />
+            </visual>
+            <!-- Right Track: Front Nose Cap -->
+            <visual>
+                <origin xyz="${sprocket_x} ${-track_y_offset} ${sprocket_z}" rpy="${PI/2} 0 0" />
+                <geometry>
+                    <cylinder radius="${sprocket_radius + 0.002}" length="${track_width}" />
+                </geometry>
+                <material name="tread_dark" />
+            </visual>
+            <!-- Right Track: Rear Tail Cap -->
+            <visual>
+                <origin xyz="${-sprocket_x} ${-track_y_offset} ${sprocket_z}" rpy="${PI/2} 0 0" />
+                <geometry>
+                    <cylinder radius="${sprocket_radius + 0.002}" length="${track_width}" />
+                </geometry>
+                <material name="tread_dark" />
+            </visual>
+            <!-- Right Track: Cleats / Grousers on Top Belt -->
+            <visual><origin xyz="-0.120 ${-track_y_offset} ${sprocket_z + sprocket_radius + 0.002}" rpy="0 0 0" /><geometry><box size="0.008 ${track_width + 0.002} 0.004" /></geometry><material name="black" /></visual>
+            <visual><origin xyz="-0.085 ${-track_y_offset} ${sprocket_z + sprocket_radius + 0.002}" rpy="0 0 0" /><geometry><box size="0.008 ${track_width + 0.002} 0.004" /></geometry><material name="black" /></visual>
+            <visual><origin xyz="-0.050 ${-track_y_offset} ${sprocket_z + sprocket_radius + 0.002}" rpy="0 0 0" /><geometry><box size="0.008 ${track_width + 0.002} 0.004" /></geometry><material name="black" /></visual>
+            <visual><origin xyz="-0.017 ${-track_y_offset} ${sprocket_z + sprocket_radius + 0.002}" rpy="0 0 0" /><geometry><box size="0.008 ${track_width + 0.002} 0.004" /></geometry><material name="black" /></visual>
+            <visual><origin xyz="0.017 ${-track_y_offset} ${sprocket_z + sprocket_radius + 0.002}" rpy="0 0 0" /><geometry><box size="0.008 ${track_width + 0.002} 0.004" /></geometry><material name="black" /></visual>
+            <visual><origin xyz="0.050 ${-track_y_offset} ${sprocket_z + sprocket_radius + 0.002}" rpy="0 0 0" /><geometry><box size="0.008 ${track_width + 0.002} 0.004" /></geometry><material name="black" /></visual>
+            <visual><origin xyz="0.085 ${-track_y_offset} ${sprocket_z + sprocket_radius + 0.002}" rpy="0 0 0" /><geometry><box size="0.008 ${track_width + 0.002} 0.004" /></geometry><material name="black" /></visual>
+            <visual><origin xyz="0.120 ${-track_y_offset} ${sprocket_z + sprocket_radius + 0.002}" rpy="0 0 0" /><geometry><box size="0.008 ${track_width + 0.002} 0.004" /></geometry><material name="black" /></visual>
+            <!-- Right Track: Mudguard / Fender -->
+            <visual>
+                <origin xyz="0.0 ${-track_y_offset} 0.060" rpy="0 0 0" />
+                <geometry>
+                    <box size="0.300 ${track_width + 0.010} 0.004" />
+                </geometry>
+                <material name="mid_grey" />
+            </visual>
+            <visual>
+                <origin xyz="0.165 ${-track_y_offset} 0.050" rpy="0 0.50 0" />
+                <geometry>
+                    <box size="0.045 ${track_width + 0.010} 0.004" />
+                </geometry>
+                <material name="mid_grey" />
+            </visual>
+            <visual>
+                <origin xyz="-0.165 ${-track_y_offset} 0.050" rpy="0 -0.50 0" />
+                <geometry>
+                    <box size="0.045 ${track_width + 0.010} 0.004" />
+                </geometry>
+                <material name="mid_grey" />
+            </visual>
+            <visual>
+                <origin xyz="0.0 ${-(track_y_offset + track_width/2 + 0.004)} 0.048" rpy="0 0 0" />
+                <geometry>
+                    <box size="0.280 0.003 0.020" />
+                </geometry>
+                <material name="mid_grey" />
+            </visual>
+            <!-- Chassis Collision (raised to avoid dragging on ground or ramps) -->
             <collision>
-                <origin xyz="0.0 0.0 ${base_z/2}" rpy="0 0 0" />
-                <geometry>
-                    <box size="${base_x} ${base_y} ${base_z}" />
+                <origin xyz="0.0 0.0 ${base_z/2 + 0.005}" rpy="0 0 0" />
+                <geometry>
+                    <box size="${base_x - 0.02} ${base_y} ${base_z - 0.01}" />
                 </geometry>
             </collision>
             <inertial>
-                <origin xyz="0.0 0.0 ${base_z/2}" rpy="0 0 0" />
+                <origin xyz="0.0 0.0 0.01" rpy="0 0 0" />
                 <mass value="${base_mass}" />
                 <inertia ixx="${(1.0/12.0)*base_mass*(base_y*base_y + base_z*base_z)}"
-                                 ixy="0.0" ixz="0.0"
-                                 iyy="${(1.0/12.0)*base_mass*(base_x*base_x + base_z*base_z)}"
-                                 iyz="0.0"
-                                 izz="${(1.0/12.0)*base_mass*(base_x*base_x + base_y*base_y)}" />
+                         ixy="0.0" ixz="0.0"
+                         iyy="${(1.0/12.0)*base_mass*(base_x*base_x + base_z*base_z)}"
+                         iyz="0.0"
+                         izz="${(1.0/12.0)*base_mass*(base_x*base_x + base_y*base_y)}" />
             </inertial>
         </link>
-        <xacro:macro name="wheel" params="prefix y_reflect">
-            <link name="wheel_${prefix}_link">
+        <!-- ================= MACRO: TANK ROAD WHEEL ================= -->
+        <xacro:macro name="road_wheel" params="prefix suffix x_pos y_reflect">
+            <link name="wheel_${prefix}_${suffix}_link">
+                <!-- Outer Rubber Roller Wheel -->
                 <visual>
                     <origin xyz="0 0 0" rpy="${PI/2} 0 0" />
                     <geometry>
-                        <cylinder radius="${wheel_radius}" length="${wheel_width}" />
+                        <cylinder radius="${road_radius}" length="${road_width - 0.004}" />
+                    </geometry>
+                    <material name="tread_dark" />
+                </visual>
+                <!-- Metallic Wheel Rim Disc (High Contrast) -->
+                <visual>
+                    <origin xyz="0 ${y_reflect * (road_width/2 - 0.001)} 0" rpy="${PI/2} 0 0" />
+                    <geometry>
+                        <cylinder radius="${road_radius * 0.78}" length="0.003" />
+                    </geometry>
+                    <material name="light_grey" />
+                </visual>
+                <!-- Tank Wheel Hubcap (Outer face) -->
+                <visual>
+                    <origin xyz="0 ${y_reflect * (road_width/2 + 0.001)} 0" rpy="${PI/2} 0 0" />
+                    <geometry>
+                        <cylinder radius="${road_radius * 0.45}" length="0.003" />
+                    </geometry>
+                    <material name="accent_orange" />
+                </visual>
+                <!-- Central Axle Bolt -->
+                <visual>
+                    <origin xyz="0 ${y_reflect * (road_width/2 + 0.003)} 0" rpy="${PI/2} 0 0" />
+                    <geometry>
+                        <cylinder radius="${road_radius * 0.18}" length="0.002" />
                     </geometry>
                     <material name="black" />
@@ -68,68 +291,111 @@
                     <origin xyz="0 0 0" rpy="${PI/2} 0 0" />
                     <geometry>
-                        <cylinder radius="${wheel_radius}" length="${wheel_width}" />
+                        <cylinder radius="${road_radius}" length="${road_width}" />
                     </geometry>
                 </collision>
                 <inertial>
                     <origin xyz="0 0 0" />
-                    <mass value="${wheel_mass}" />
-                    <inertia ixx="${(1.0/12.0)*wheel_mass*(3*wheel_radius*wheel_radius + wheel_width*wheel_width)}"
-                                     ixy="0" ixz="0"
-                                     iyy="${(1.0/12.0)*wheel_mass*(3*wheel_radius*wheel_radius + wheel_width*wheel_width)}"
-                                     iyz="0"
-                                     izz="${(1.0/2.0)*wheel_mass*wheel_radius*wheel_radius}" />
+                    <mass value="${road_mass}" />
+                    <inertia ixx="${(1.0/12.0)*road_mass*(3*road_radius*road_radius + road_width*road_width)}"
+                             ixy="0" ixz="0"
+                             iyy="${(1.0/12.0)*road_mass*(3*road_radius*road_radius + road_width*road_width)}"
+                             iyz="0"
+                             izz="${(1.0/2.0)*road_mass*road_radius*road_radius}" />
                 </inertial>
             </link>
-            <joint name="wheel_${prefix}_joint" type="continuous">
+            <joint name="wheel_${prefix}_${suffix}_joint" type="continuous">
                 <parent link="base_link" />
-                <child link="wheel_${prefix}_link" />
-                <origin xyz="${wheel_x_offset} ${y_reflect * wheel_separation/2} 0.0" rpy="0 0 0" />
+                <child link="wheel_${prefix}_${suffix}_link" />
+                <origin xyz="${x_pos} ${y_reflect * track_y_offset} 0.0" rpy="0 0 0" />
                 <axis xyz="0 1 0" />
-                <dynamics damping="0.01" friction="0.1" />
+                <dynamics damping="0.01" friction="0.05" />
             </joint>
+            <gazebo reference="wheel_${prefix}_${suffix}_link">
+                <mu1>1.5</mu1>
+                <mu2>0.1</mu2>
+                <kp>1000000.0</kp>
+                <kd>1.0</kd>
+                <minDepth>0.001</minDepth>
+            </gazebo>
         </xacro:macro>
-        <xacro:wheel prefix="left" y_reflect="1" />
-        <xacro:wheel prefix="right" y_reflect="-1" />
-        <xacro:macro name="caster" params="prefix x_offset">
-            <link name="caster_${prefix}_link">
-                <visual>
-                    <origin xyz="0 0 0" rpy="0 0 0" />
-                    <geometry>
-                        <sphere radius="${caster_radius}" />
+        <!-- ================= MACRO: SPROCKET / IDLER WHEEL ================= -->
+        <xacro:macro name="end_wheel" params="type prefix x_pos z_pos y_reflect">
+            <link name="${type}_${prefix}_link">
+                <!-- Sprocket / Idler Wheel Body -->
+                <visual>
+                    <origin xyz="0 0 0" rpy="${PI/2} 0 0" />
+                    <geometry>
+                        <cylinder radius="${sprocket_radius}" length="${sprocket_width - 0.004}" />
+                    </geometry>
+                    <material name="tread_dark" />
+                </visual>
+                <!-- Metallic Wheel Rim Disc -->
+                <visual>
+                    <origin xyz="0 ${y_reflect * (sprocket_width/2 - 0.001)} 0" rpy="${PI/2} 0 0" />
+                    <geometry>
+                        <cylinder radius="${sprocket_radius * 0.78}" length="0.003" />
+                    </geometry>
+                    <material name="light_grey" />
+                </visual>
+                <!-- Outer Hubcap -->
+                <visual>
+                    <origin xyz="0 ${y_reflect * (sprocket_width/2 + 0.001)} 0" rpy="${PI/2} 0 0" />
+                    <geometry>
+                        <cylinder radius="${sprocket_radius * 0.45}" length="0.003" />
+                    </geometry>
+                    <material name="accent_orange" />
+                </visual>
+                <visual>
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